File: eload.kicad_pcb (KiCad board)
At the start: 2 copper layers, 78.7 x 99.1 mm, 62 parts, among them J1 Device Power, J2 Input, J3 JST Header, J4 SWD Header, J6 JST Header, J7 Conn_02x06_Odd_Even, K1 G5Q-1, Q1 RFP30N06LE-VB, Q2 HL 40N05, Q3 DTC043ZUBTL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

Commit message: PCB Routing
Parts:
- added J5: Conn_01x08_Socket, Connector_JST:JST_XH_B8B-XH-A_1x08_P2.50mm_Vertical, F.Cu at (76.2, 93.8)
- added J8: Conn_01x08_Socket, Connector_JST:JST_XH_B8B-XH-A_1x08_P2.50mm_Vertical, F.Cu at (81.6, 163.6)
- TP2: footprint TestPoint:TestPoint_Pad_D1.5mm -> TestPoint:TestPoint_Loop_D1.80mm_Drill1.0mm_Beaded
- moved J7 60.7 mm to (26.4, 88.1)
- moved J4 56.8 mm to (84.3, 95.5), turned to 0 degrees
- moved TP2 32.5 mm to (91.4, 80.8)
- moved H3 31.2 mm to (19.1, 114.8)
- moved H4 31.2 mm to (90.2, 114.8)
- moved D2 25.2 mm to (44.7, 72.3), turned to -90 degrees
- moved TP3 21.9 mm to (41.7, 69.6)
- moved K1 18.9 mm to (48.3, 76.4), turned to 0 degrees
- moved TP1 18.7 mm to (90.2, 85.9)
- moved J3 16.9 mm to (29.9, 110.5)
- moved Q2 13.9 mm to (51.6, 81.0), turned to 90 degrees
- moved F1 12.1 mm to (54.4, 65.0), turned to 0 degrees
- moved R5 9.15 mm to (57.1, 85.4)
- moved R6 7.91 mm to (56.1, 90.4), turned to 180 degrees
- moved C3 7.87 mm to (51.1, 98.3), turned to 180 degrees
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Connections:
- J3 pad 10: /D0 -> /D3
- J3 pad 11: /D1 -> /D4
- J3 pad 12: /D2 -> /D5
- J3 pad 13: /D3 -> /D6
- J3 pad 14: /D4 -> /D7
- J3 pad 15: /D5 -> +3.3V
- J3 pad 16: /D6 -> GND
- J3 pad 2: /EncB -> +3.3V
- J3 pad 3: /EncA -> /Interface/V0
- J3 pad 4: /EncSw -> /RS
- J3 pad 5: unconnected-(J3-Pin_5-Pad5) -> GND
- J3 pad 6: /OvDetect -> /E
- J3 pad 7: /LoadEn -> /D0
- J3 pad 8: /RS -> /D1
- J3 pad 9: /E -> /D2
- J6 pad 10: /D0 -> /D3
- J6 pad 11: /D1 -> /D4
- J6 pad 12: /D2 -> /D5
- J6 pad 13: /D3 -> /D6
- J6 pad 14: /D4 -> /D7
- J6 pad 15: /D5 -> +3.3V
- J6 pad 16: /D6 -> GND
- J6 pad 2: /EncB -> +3.3V
- J6 pad 3: /EncA -> /Interface/V0
- J6 pad 4: /EncSw -> /RS
- J6 pad 5: unconnected-(J6-Pin_5-Pad5) -> GND
- J6 pad 6: /OvDetect -> /E
- J6 pad 7: /LoadEn -> /D0
- J6 pad 8: /RS -> /D1
- J6 pad 9: /E -> /D2
- J7 pad 11: /PB1 -> +3.3V
- Q1 pad 1: Net-(Q1-G) -> /Isense
- U2 pad 19: /PB1 -> /Isense
- U2 pad 31: /LoadEn -> /OvDetect
- U2 pad 32: /OvDetect -> /LoadEn
- U3 pad 1: Net-(Q1-G) -> /Isense
Routing:
- net +3.3V: track 22.2 -> 217.9 mm
- net /Isense: track 0.00 -> 79.1 mm
- net +5V: track 28.8 -> 83.5 mm
- net /RS: track 0.00 -> 50.9 mm, vias 0 -> 2
- net /LoadEn: track 0.00 -> 48.0 mm, vias 0 -> 4
- net /E: track 0.00 -> 42.2 mm, vias 0 -> 2
- net /SCL: track 0.00 -> 40.1 mm
- net /SDA: track 0.00 -> 35.7 mm
- net /D0: track 0.00 -> 20.2 mm
- net /D1: track 0.00 -> 17.7 mm
- net /D2: track 0.00 -> 14.5 mm
- net /EncSw: track 0.00 -> 14.5 mm
- net /VCC_sense: track 0.00 -> 13.9 mm
- net /EncA: track 0.00 -> 13.6 mm
- net /EncB: track 0.00 -> 13.3 mm
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Other:
- board size 78.7 x 99.1 mm -> 78.7 x 67.6 mm
